File: hardware/ram-pak/hyperram.sch (KiCad schematic (older format))
At the start: 4 parts, among them U2 S70KL1281

Commit message: ram-pak: silkscreen improvements.
Changed lines of the file:
@@
 $Descr A4 11693 8268
 encoding utf-8
-Sheet 2 3
+Sheet 3 3
 Title "iCEBreaker PMOD - Hyperram"
 Date ""
@@
 AR Path="/60051CB7/5E0FA7AE" Ref="U3"  Part="1"
 AR Path="/60051CE0/5E0FA7AE" Ref="U?"  Part="1"
-F 0 "U2" H 5600 3680 50  0000 C CNN
+F 0 "U3" H 5600 3680 50  0000 C CNN
 F 1 "S70KL1281" H 5600 3587 50  0000 C CNN
 F 2 "pkl_housings_bga:BGA-24_5x5_6.0x8.0mm" H 6200 1850 50  0001 C CNN
@@
 AR Path="/60051CB7/5E0FA7CA" Ref="#PWR013"  Part="1"
 AR Path="/60051CE0/5E0FA7CA" Ref="#PWR?"  Part="1"
-F 0 "#PWR09" H 4900 3400 50  0001 C CNN
+F 0 "#PWR013" H 4900 3400 50  0001 C CNN
 F 1 "GND" H 4905 3474 50  0000 C CNN
 F 2 "" H 4900 3650 50  0001 C CNN
@@
 AR Path="/60051CB7/5E0FA7EE" Ref="C8"  Part="1"
 AR Path="/60051CE0/5E0FA7EE" Ref="C?"  Part="1"
-F 0 "C5" H 5342 4097 50  0000 L CNN
+F 0 "C8" H 5342 4097 50  0000 L CNN
 F 1 "100n" H 5342 4004 50  0000 L CNN
 F 2 "pkl_dipol:C_0402" H 5342 3957 60  0001 L CNN
@@
 AR Path="/60051CB7/5E0FA7F5" Ref="C9"  Part="1"
 AR Path="/60051CE0/5E0FA7F5" Ref="C?"  Part="1"
-F 0 "C6" H 5642 4097 50  0000 L CNN
+F 0 "C9" H 5642 4097 50  0000 L CNN
 F 1 "100n" H 5642 4004 50  0000 L CNN
 F 2 "pkl_dipol:C_0402" H 5550 4050 60  0001 C CNN
@@
 AR Path="/60051CB7/5E0FA7FC" Ref="C10"  Part="1"
 AR Path="/60051CE0/5E0FA7FC" Ref="C?"  Part="1"
-F 0 "C7" H 5942 4097 50  0000 L CNN
+F 0 "C10" H 5942 4097 50  0000 L CNN
 F 1 "100n" H 5942 4004 50  0000 L CNN
 F 2 "pkl_dipol:C_0402" H 5850 4050 60  0001 C CNN
@@
 AR Path="/60051CB7/5E0FA810" Ref="#PWR015"  Part="1"
 AR Path="/60051CE0/5E0FA810" Ref="#PWR?"  Part="1"
-F 0 "#PWR011" H 5550 4100 50  0001 C CNN
+F 0 "#PWR015" H 5550 4100 50  0001 C CNN
 F 1 "GND" H 5555 4174 50  0000 C CNN
 F 2 "" H 5550 4350 50  0001 C CNN
@@
 AR Path="/60051C8E/6001E263" Ref="#PWR?"  Part="1"
 AR Path="/60051CE0/6001E263" Ref="#PWR?"  Part="1"
-F 0 "#PWR08" H 4900 1700 50  0001 C CNN
+F 0 "#PWR012" H 4900 1700 50  0001 C CNN
 F 1 "+1V8" H 4915 2023 50  0000 C CNN
 F 2 "" H 4900 1850 50  0001 C CNN
@@
 AR Path="/60051C8E/6003ACB3" Ref="#PWR?"  Part="1"
 AR Path="/60051CE0/6003ACB3" Ref="#PWR?"  Part="1"
-F 0 "#PWR010" H 5550 3600 50  0001 C CNN
+F 0 "#PWR014" H 5550 3600 50  0001 C CNN
 F 1 "+1V8" H 5565 3923 50  0000 C CNN
 F 2 "" H 5550 3750 50  0001 C CNN

Commit message: ram-pak: Extended and updated BOM information.
Parts:
- C5, C6, C7: 1b2-bom-key (none) -> cap-cer-0402-100n
- U2: value S70KL1281 -> W957D8MFYA5I; 1b2-bom-key (none) -> ram-24vbga-w957d8mfya5i
Changed lines of the file:
@@
 AR Path="/60051CE0/5E0FA7AE" Ref="U?"  Part="1"
 F 0 "U3" H 5600 3680 50  0000 C CNN
-F 1 "S70KL1281" H 5600 3587 50  0000 C CNN
+F 1 "W957D8MFYA5I" H 5600 3587 50  0000 C CNN
 F 2 "pkl_housings_bga:BGA-24_5x5_6.0x8.0mm" H 6200 1850 50  0001 C CNN
-F 3 "http://www.cypress.com/file/183506/download" H 5600 1850 50  0001 C CNN
+F 3 "https://www.mouser.com/datasheet/2/949/W957x8MFYA_128Mb_HyperRAM_TFBGA24_DDP_datasheet_A0-1928530.pdf" H 5600 1850 50  0001 C CNN
 F 4 "ANY" H 5600 2750 50  0001 C CNN "Source"
+F 5 "ram-24vbga-w957d8mfya5i" H 5600 2750 50  0001 C CNN "1b2-bom-key"
 	1    5600 2750
 	1    0    0    -1
@@
 F 3 "" H 5250 4050 60  0000 C CNN
 F 4 "ANY" H 5250 4050 50  0001 C CNN "Source"
+F 5 "cap-cer-0402-100n" H 5250 4050 50  0001 C CNN "1b2-bom-key"
 	1    5250 4050
 	1    0    0    -1
@@
 F 3 "" H 5550 4050 60  0000 C CNN
 F 4 "ANY" H 5550 4050 50  0001 C CNN "Source"
+F 5 "cap-cer-0402-100n" H 5550 4050 50  0001 C CNN "1b2-bom-key"
 	1    5550 4050
 	1    0    0    -1
@@
 F 3 "" H 5850 4050 60  0000 C CNN
 F 4 "ANY" H 5850 4050 50  0001 C CNN "Source"
+F 5 "cap-cer-0402-100n" H 5850 4050 50  0001 C CNN "1b2-bom-key"
 	1    5850 4050
 	1    0    0    -1
